Commit message: nav working with control

File: src/qcar_gazebo/urdf/depth_camera.xacro (robot description, xacro)
@@ -25,4 +25,10 @@
             <plugin name="camera_controller" filename="libgazebo_ros_depth_camera.so">
                 <cameraName>depth_camera</cameraName>
+                <frameName>camera_rgb_optical</frameName>
+                <imageTopicName>image_raw</imageTopicName>
+                <cameraInfoTopicName>camera_info</cameraInfoTopicName>
+                <depthImageTopicName>depth/image_raw</depthImageTopicName>
+                <depthImageCameraInfoTopicName>depth/camera_info</depthImageCameraInfoTopicName>
+                <pointCloudTopicName>points</pointCloudTopicName>
             </plugin>
         </sensor>

File: src/qcar_gazebo/urdf/qcar_model.xacro (robot description, xacro)
@@ -4,5 +4,5 @@
   <xacro:include filename="$(find gazebo_ros_motors)/xacro/joint_motor.xacro"/>
   <xacro:include filename="$(find gazebo_ros_motors)/xacro/dc_motor.xacro"/> <!--dc motor plugin include-->
-  <!-- <xacro:include filename="$(find qcar_gazebo)/urdf/lidar.xacro" /> -->
+  <xacro:include filename="$(find qcar_gazebo)/urdf/lidar.xacro" />
   <xacro:include filename="$(find qcar_gazebo)/urdf/camera.xacro" />
   <xacro:include filename="$(find qcar_gazebo)/urdf/depth_camera.xacro" />
@@ -247,4 +247,10 @@
   	</joint>
     <link name="camera_rgb"/>
+    <joint name="camera_rgb_optical_joint" type="fixed">
+        <parent link="camera_rgb"/>
+        <child link="camera_rgb_optical"/>
+        <origin xyz="0 0 0" rpy="-1.5708 0 -1.5708"/>
+    </joint>
+    <link name="camera_rgb_optical"/>
     <joint name="camera_csi_front_joint" type="fixed">
         <!-- <axis xyz="0 1 0" /> -->
